Commit message: Update rugved_description.urdf

File: rugved_description/urdf/rugved_description.urdf (robot description, URDF)
Before this commit: robot rugved_description, 5 links, 4 joints
Joints:
- joint horizontal_castor_joint: limit lower=0 upper=20 effort=500 velocity=0.2 -> effort=500 velocity=0.2; type revolute -> continuous
- joint left_wheel_joint: limit lower=0 upper=20 effort=1000 velocity=0.2 -> effort=1000 velocity=0.2; type revolute -> continuous
- joint right_wheel_joint: limit lower=0 upper=20 effort=1000 velocity=0.2 -> effort=1000 velocity=0.2; type revolute -> continuous
- joint vertical_castor_joint: limit lower=0 upper=20 effort=400 velocity=0.2 -> effort=400 velocity=0.2; type revolute -> continuous

Commit message: Update rugved_description.urdf

File: rugved_description/urdf/rugved_description.urdf (robot description, URDF)
Before this commit: robot rugved_description, 5 links, 4 joints
Links:
- added link hokuyo_link, mass 1e-5; collision box size=0.1 0.1 0.1; visual box size=0.1 0.1 0.1
Joints:
- added joint hokuyo_joint: type fixed, parent base_link, child hokuyo_link, origin xyz=-0.56 0 0.56 rpy=0 0 3.141, axis 0 1 0
- joint horizontal_castor_joint: limit effort=500 velocity=0.2 -> lower=0 upper=20 effort=500 velocity=0.2; type continuous -> revolute
- joint left_wheel_joint: limit effort=1000 velocity=0.2 -> lower=0 upper=20 effort=1000 velocity=0.2; type continuous -> revolute
- joint right_wheel_joint: limit effort=1000 velocity=0.2 -> lower=0 upper=20 effort=1000 velocity=0.2; type continuous -> revolute
- joint vertical_castor_joint: limit effort=400 velocity=0.2 -> lower=0 upper=20 effort=400 velocity=0.2; type continuous -> revolute
